File: exodia_stage_hand_clinical/hardware/kicad/wrist_pcb/wrist_pcb.kicad_sch (KiCad schematic)
At the start: 11 parts, among them J1 USB_C_CHARGE_IN, J2 ZIF_5PIN_FLEX_HARNESS, Q1 IRLZ44N_HEATER, Q2 2N7002_IDX, Q3 2N7002_MID, Q4 2N7002_RNG, Q5 2N7002_PNK, U1 ESP32-S3-MINI-1, U2 TP4056

Commit message: Replace schematic with minimal working template and add component checklist
Parts:
- removed J1: USB_C_CHARGE_IN, symbol USBC_CONN
- removed J2: ZIF_5PIN_FLEX_HARNESS, symbol ZIF_5PIN
- removed Q1: IRLZ44N_HEATER, symbol IRLZ44N_MOSFET
- removed Q2: 2N7002_IDX, symbol 2N7002_MOSFET
- removed Q3: 2N7002_MID, symbol 2N7002_MOSFET
- removed Q4: 2N7002_RNG, symbol 2N7002_MOSFET
- removed Q5: 2N7002_PNK, symbol 2N7002_MOSFET
- removed R1: 10K, symbol R_FIXED
- removed RT1: NTC_10K_B3950, symbol NTC_THERMISTOR
- removed U1: ESP32-S3-MINI-1, symbol ESP32S3_MODULE
- removed U2: TP4056, symbol TP4056_IC
Other:
- note removed: "ALL JOINTS: Apply MG Chemicals 422B conformal coat after assembly. Cure 30 min minimum."
- note removed: "THERMAL SAFETY: Firmware cutoff at 40C NTC sensor fail = heater OFF BLE timeout 30s = all OFF"
- note removed: "ZIF J2 -> Flex Finger Harness (1-layer polyimide, coverlay both sides) Bond harness to glove with 3M 9485PC tape."
Changed lines of the file:
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@@
     (rev "v1.0")
     (company "Resonanx")
-    (comment 1 "Memory Care Edition — Single ESP32-S3, Rigid+Flex split")
+    (comment 1 "Memory Care Edition — Single ESP32-S3")
     (comment 2 "Board 1 of 2: Rigid Wrist PCB")
   )
-  (symbol (lib_id "USBC_CONN") (at 25 170 0) (unit 1)
-    (property "Reference" "J1" (at 25 163 0))
-    (property "Value" "USB_C_CHARGE_IN" (at 25 177 0))
-  )
-  (symbol (lib_id "TP4056_IC") (at 55 170 0) (unit 1)
-    (property "Reference" "U2" (at 55 163 0))
-    (property "Value" "TP4056" (at 55 177 0))
-  )
-  (symbol (lib_id "PWR_FLAG") (at 80 155 0) (unit 1)
-    (property "Reference" "#PWR01" (at 80 152 0))
-    (property "Value" "VBAT_SW" (at 80 158 0))
-  )
-  (symbol (lib_id "ESP32S3_MODULE") (at 120 130 0) (unit 1)
-    (property "Reference" "U1" (at 120 120 0))
-    (property "Value" "ESP32-S3-MINI-1" (at 120 142 0))
-  )
-  (symbol (lib_id "IRLZ44N_MOSFET") (at 165 100 0) (unit 1)
-    (property "Reference" "Q1" (at 165 95 0))
-    (property "Value" "IRLZ44N_HEATER" (at 165 107 0))
-  )
-  (symbol (lib_id "2N7002_MOSFET") (at 165 120 0) (unit 1)
-    (property "Reference" "Q2" (at 165 115 0))
-    (property "Value" "2N7002_IDX" (at 165 127 0))
-  )
-  (symbol (lib_id "2N7002_MOSFET") (at 165 135 0) (unit 1)
-    (property "Reference" "Q3" (at 165 130 0))
-    (property "Value" "2N7002_MID" (at 165 142 0))
-  )
-  (symbol (lib_id "2N7002_MOSFET") (at 165 150 0) (unit 1)
-    (property "Reference" "Q4" (at 165 145 0))
-    (property "Value" "2N7002_RNG" (at 165 157 0))
-  )
-  (symbol (lib_id "2N7002_MOSFET") (at 165 165 0) (unit 1)
-    (property "Reference" "Q5" (at 165 160 0))
-    (property "Value" "2N7002_PNK" (at 165 172 0))
-  )
-  (symbol (lib_id "R_FIXED") (at 85 100 0) (unit 1)
-    (property "Reference" "R1" (at 82 100 0))
-    (property "Value" "10K" (at 88 100 0))
-  )
-  (symbol (lib_id "NTC_THERMISTOR") (at 85 110 0) (unit 1)
-    (property "Reference" "RT1" (at 82 110 0))
-    (property "Value" "NTC_10K_B3950" (at 88 110 0))
-  )
-  (symbol (lib_id "ZIF_5PIN") (at 200 130 0) (unit 1)
-    (property "Reference" "J2" (at 200 122 0))
-    (property "Value" "ZIF_5PIN_FLEX_HARNESS" (at 200 140 0))
-  )
-  (symbol (lib_id "VCC") (at 80 148 0) (unit 1)
-    (property "Reference" "#PWR02" (at 80 148 0) (effects (hide yes)))
-    (property "Value" "VCC" (at 80 145 0))
-  )
-  (symbol (lib_id "GND") (at 120 185 0) (unit 1)
-    (property "Reference" "#PWR03" (at 120 185 0) (effects (hide yes)))
-    (property "Value" "GND" (at 120 188 0))
-  )
-  (wire (pts (xy 31 170) (xy 47 170)))
-  (wire (pts (xy 63 168) (xy 80 168) (xy 80 152)))
-  (wire (pts (xy 80 152) (xy 110 130)))
-  (wire (pts (xy 110 126) (xy 159 100)))
-  (wire (pts (xy 110 122) (xy 159 120)))
-  (wire (pts (xy 110 120) (xy 159 135)))
-  (wire (pts (xy 110 118) (xy 159 150)))
-  (wire (pts (xy 110 116) (xy 159 165)))
-  (wire (pts (xy 110 128) (xy 90 115) (xy 90 110)))
-  (wire (pts (xy 85 95) (xy 85 90)))
-  (wire (pts (xy 85 90) (xy 80 90) (xy 80 152)))
-  (wire (pts (xy 85 115) (xy 85 120) (xy 120 120) (xy 120 185)))
-  (wire (pts (xy 171 98) (xy 194 128)))
-  (wire (pts (xy 171 118) (xy 194 126)))
-  (wire (pts (xy 171 133) (xy 194 124)))
-  (wire (pts (xy 171 148) (xy 194 122)))
-  (wire (pts (xy 171 163) (xy 194 120)))
-  (wire (pts (xy 80 152) (xy 194 132)))
-  (wire (pts (xy 171 102) (xy 171 185) (xy 120 185)))
-  (wire (pts (xy 171 122) (xy 171 185)))
-  (wire (pts (xy 171 137) (xy 171 185)))
-  (wire (pts (xy 171 152) (xy 171 185)))
-  (wire (pts (xy 171 167) (xy 171 185)))
-  (wire (pts (xy 25 174) (xy 25 185) (xy 120 185)))
-  (label "HEATER_PWM" (at 130 126 0) (effects (font (size 1.27 1.27))))
-  (label "MOTOR_IDX_PWM" (at 130 122 0) (effects (font (size 1.27 1.27))))
-  (label "MOTOR_MID_PWM" (at 130 120 0) (effects (font (size 1.27 1.27))))
-  (label "MOTOR_RNG_PWM" (at 130 118 0) (effects (font (size 1.27 1.27))))
-  (label "MOTOR_PNK_PWM" (at 130 116 0) (effects (font (size 1.27 1.27))))
-  (label "NTC_ADC" (at 105 128 0) (effects (font (size 1.27 1.27))))
-  (label "TO_FLEX_HARNESS" (at 208 130 0) (effects (font (size 1.27 1.27))))
-  (text "THERMAL SAFETY:\nFirmware cutoff at 40C\nNTC sensor fail = heater OFF\nBLE timeout 30s = all OFF"
-    (at 20 100 0) (effects (font (size 1.27 1.27)) (justify left)))
-  (text "ALL JOINTS: Apply MG Chemicals 422B\nconformal coat after assembly.\nCure 30 min minimum."
-    (at 20 115 0) (effects (font (size 1.27 1.27)) (justify left)))
-  (text "ZIF J2 -> Flex Finger Harness\n(1-layer polyimide, coverlay both sides)\nBond harness to glove with 3M 9485PC tape."
-    (at 210 120 0) (effects (font (size 1.27 1.27)) (justify left)))
 )
